File: kicad/xbox_1.6/xbox_1.6.kicad_pcb (KiCad board)
At the start: 2 copper layers, 6 parts, among them U2C1 intel_495_bga2, U4B1 ddr_100_tqfp, U4C1 nvidia_xgpu_nv2a, U5F1 ddr_100_tqfp, U6D1 ddr_100_tqfp, U6E1 nvidia_mcpx

Commit message: route more traces
Connections:
- net CPU_D23 renamed /CPU_D23
- net CPU_D33 renamed /CPU_D33
- net CPU_D35 renamed /CPU_D35
- U2C1 pad D19: (no net) -> /CPU_D32
- U2C1 pad D20: (no net) -> /CPU_D37
- U2C1 pad D21: (no net) -> /CPU_D38
- U2C1 pad F19: (no net) -> /CPU_D36
Routing:
- net /CPU_D37: track 0.00 -> 1.37 mm, vias 0 -> 1
- net /CPU_D38: track 0.00 -> 1.26 mm, vias 0 -> 1
- net /CPU_D32: track 0.00 -> 0.88 mm, vias 0 -> 1
- net /CPU_D36: track 0.00 -> 0.87 mm, vias 0 -> 1
Changed lines of the file:
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@@
   (net 5 "/CPU_D21")
   (net 6 "/CPU_D27")
-  (net 7 "CPU_D23")
-  (net 8 "CPU_D33")
-  (net 9 "CPU_D35")
+  (net 7 "/CPU_D23")
+  (net 8 "/CPU_D33")
+  (net 9 "/CPU_D35")
+  (net 10 "/CPU_D38")
+  (net 11 "/CPU_D37")
+  (net 12 "/CPU_D32")
+  (net 13 "/CPU_D36")
   (footprint "xbox_footprint:intel_495_bga2" (layer "F.Cu")
     (at 275.145 116.76)
@@
     (pad "A17" smd circle (at -14.605 -7.62 90) (size 0.55 0.55) (layers "F.Cu" "F.Paste" "F.Mask"))
     (pad "A18" smd circle (at -14.605 -8.89 90) (size 0.55 0.55) (layers "F.Cu" "F.Paste" "F.Mask")
-      (net 7 "CPU_D23"))
+      (net 7 "/CPU_D23"))
     (pad "A19" smd circle (at -14.605 -10.16 90) (size 0.55 0.55) (layers "F.Cu" "F.Paste" "F.Mask")
       (net 5 "/CPU_D21"))
@@
       (net 4 "/VSS"))
     (pad "C20" smd circle (at -12.065 -11.43 90) (size 0.55 0.55) (layers "F.Cu" "F.Paste" "F.Mask")
-      (net 9 "CPU_D35"))
+      (net 9 "/CPU_D35"))
     (pad "C21" smd circle (at -12.065 -12.7 90) (size 0.55 0.55) (layers "F.Cu" "F.Paste" "F.Mask")
-      (net 8 "CPU_D33"))
+      (net 8 "/CPU_D33"))
     (pad "D1" smd circle (at -10.795 12.7 90) (size 0.55 0.55) (layers "F.Cu" "F.Paste" "F.Mask"))
     (pad "D2" smd circle (at -10.795 11.43 90) (size 0.55 0.55) (layers "F.Cu" "F.Paste" "F.Mask"))
@@
     (pad "D17" smd circle (at -10.795 -7.62 90) (size 0.55 0.55) (layers "F.Cu" "F.Paste" "F.Mask"))
     (pad "D18" smd circle (at -10.795 -8.89 90) (size 0.55 0.55) (layers "F.Cu" "F.Paste" "F.Mask"))
-    (pad "D19" smd circle (at -10.795 -10.16 90) (size 0.55 0.55) (layers "F.Cu" "F.Paste" "F.Mask"))
-    (pad "D20" smd circle (at -10.795 -11.43 90) (size 0.55 0.55) (layers "F.Cu" "F.Paste" "F.Mask"))
-    (pad "D21" smd circle (at -10.795 -12.7 90) (size 0.55 0.55) (layers "F.Cu" "F.Paste" "F.Mask"))
+    (pad "D19" smd circle (at -10.795 -10.16 90) (size 0.55 0.55) (layers "F.Cu" "F.Paste" "F.Mask")
+      (net 12 "/CPU_D32"))
+    (pad "D20" smd circle (at -10.795 -11.43 90) (size 0.55 0.55) (layers "F.Cu" "F.Paste" "F.Mask")
+      (net 11 "/CPU_D37"))
+    (pad "D21" smd circle (at -10.795 -12.7 90) (size 0.55 0.55) (layers "F.Cu" "F.Paste" "F.Mask")
+      (net 10 "/CPU_D38"))
     (pad "E1" smd circle (at -9.525 12.7 90) (size 0.55 0.55) (layers "F.Cu" "F.Paste" "F.Mask"))
     (pad "E2" smd circle (at -9.525 11.43 90) (size 0.55 0.55) (layers "F.Cu" "F.Paste" "F.Mask"))
@@
     (pad "F17" smd circle (at -8.255 -7.62 90) (size 0.55 0.55) (layers "F.Cu" "F.Paste" "F.Mask"))
     (pad "F18" smd circle (at -8.255 -8.89 90) (size 0.55 0.55) (layers "F.Cu" "F.Paste" "F.Mask"))
-    (pad "F19" smd circle (at -8.255 -10.16 90) (size 0.55 0.55) (layers "F.Cu" "F.Paste" "F.Mask"))
+    (pad "F19" smd circle (at -8.255 -10.16 90) (size 0.55 0.55) (layers "F.Cu" "F.Paste" "F.Mask")
+      (net 13 "/CPU_D36"))
     (pad "F20" smd circle (at -8.255 -11.43 90) (size 0.55 0.55) (layers "F.Cu" "F.Paste" "F.Mask")
       (net 4 "/VSS"))
@@
   (segment (start 263.08 105.33) (end 263.08 105.35) (width 0.1) (layer "F.Cu") (net 9))
   (via (at 262.47 105.96) (size 0.56) (drill 0.3) (layers "F.Cu" "B.Cu") (net 9))
+  (segment (start 263.78 104.06) (end 263.66 104.18) (width 0.1) (layer "F.Cu") (net 10))
+  (segment (start 263.66 104.18) (end 263.66 104.7) (width 0.1) (layer "F.Cu") (net 10))
+  (segment (start 264.35 104.06) (end 263.78 104.06) (width 0.1) (layer "F.Cu") (net 10))
+  (via (at 263.66 104.7) (size 0.56) (drill 0.3) (layers "F.Cu" "B.Cu") (net 10))
+  (segment (start 264.35 105.33) (end 264.39 105.29) (width 0.1) (layer "F.Cu") (net 11))
+  (segment (start 265 104.54) (end 265.02 104.56) (width 0.1) (layer "F.Cu") (net 11))
+  (segment (start 264.51 104.54) (end 265 104.54) (width 0.1) (layer "F.Cu") (net 11))
+  (segment (start 264.39 105.29) (end 264.39 104.66) (width 0.1) (layer "F.Cu") (net 11))
+  (segment (start 264.39 104.66) (end 264.51 104.54) (width 0.1) (layer "F.Cu") (net 11))
+  (via (at 265.02 104.56) (size 0.56) (drill 0.3) (layers "F.Cu" "B.Cu") (net 11))
+  (segment (start 264.35 106.6) (end 263.73 105.98) (width 0.1) (layer "F.Cu") (net 12))
+  (via (at 263.73 105.98) (size 0.56) (drill 0.3) (layers "F.Cu" "B.Cu") (net 12))
+  (segment (start 266.89 106.6) (end 266.89 106.59) (width 0.1) (layer "F.Cu") (net 13))
+  (segment (start 266.89 106.59) (end 266.28 105.98) (width 0.1) (layer "F.Cu") (net 13))
+  (via (at 266.28 105.98) (size 0.56) (drill 0.3) (layers "F.Cu" "B.Cu") (net 13))
 )

Commit message: route more traces
Connections:
- U2C1 pad E18: (no net) -> /CPU_D34
- U2C1 pad E20: (no net) -> /CPU_D43
- U2C1 pad E21: (no net) -> /CPU_D45
- U2C1 pad F18: (no net) -> /CPU_D40
- U2C1 pad H18: (no net) -> /CPU_D39
- U2C1 pad J18: (no net) -> /CPU_D41
- U4C1 pad A4: (no net) -> /CPU_D45
Routing:
- net /CPU_D45: track 0.00 -> 79.6 mm, vias 0 -> 1
- net /CPU_D43: track 0.00 -> 19.8 mm, vias 0 -> 1
- net /CPU_D40: track 0.00 -> 1.11 mm, vias 0 -> 1
- net /CPU_D34: track 0.00 -> 1.05 mm, vias 0 -> 1
- net /CPU_D41: track 0.00 -> 0.89 mm, vias 0 -> 1
- net /CPU_D39: track 0.00 -> 0.87 mm, vias 0 -> 1

Commit message: route more
Connections:
- U4C1 pad B4: (no net) -> /CPU_D43
Routing:
- net /CPU_D43: track 19.8 -> 83.5 mm
Changed lines of the file:
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@@
     (pad "B2" smd circle (at -15.5 -15.5 270) (size 0.45 0.45) (layers "F.Cu" "F.Paste" "F.Mask"))
     (pad "B3" smd circle (at -14.5 -15.5 270) (size 0.45 0.45) (layers "F.Cu" "F.Paste" "F.Mask"))
-    (pad "B4" smd circle (at -13.5 -15.5 270) (size 0.45 0.45) (layers "F.Cu" "F.Paste" "F.Mask"))
+    (pad "B4" smd circle (at -13.5 -15.5 270) (size 0.45 0.45) (layers "F.Cu" "F.Paste" "F.Mask")
+      (net 19 "/CPU_D43"))
     (pad "B5" smd circle (at -12.5 -15.5 270) (size 0.45 0.45) (layers "F.Cu" "F.Paste" "F.Mask"))
     (pad "B6" smd circle (at -11.5 -15.5 270) (size 0.45 0.45) (layers "F.Cu" "F.Paste" "F.Mask")
@@
   (arc (start 266.7 101.83) (mid 266.65 101.71) (end 266.53 101.66) (width 0.1) (layer "F.Cu") (net 18))
   (arc (start 266.52 101.3) (mid 266.700253 101.102558) (end 266.52 100.91) (width 0.1) (layer "F.Cu") (net 18))
+  (segment (start 235.54 103.73) (end 235.7 103.89) (width 0.1) (layer "F.Cu") (net 19))
+  (segment (start 259.24 99.66) (end 259.24 99.11) (width 0.1) (layer "F.Cu") (net 19))
+  (segment (start 268.45 97.22) (end 272.07 97.22) (width 0.1) (layer "F.Cu") (net 19))
+  (segment (start 266.5 96.82) (end 266.39 96.93) (width 0.1) (layer "F.Cu") (net 19))
+  (segment (start 267.91 100.28) (end 268.11 100.28) (width 0.1) (layer "F.Cu") (net 19))
+  (segment (start 234.82 108.29) (end 234.29 108.29) (width 0.1) (layer "F.Cu") (net 19))
+  (segment (start 265.62 105.33) (end 266.27 104.68) (width 0.1) (layer "F.Cu") (net 19))
+  (segment (start 266.39 96.93) (end 266.39 98.87) (width 0.1) (layer "F.Cu") (net 19))
+  (segment (start 267.12 100.28) (end 267.12 97.35) (width 0.1) (layer "F.Cu") (net 19))
+  (segment (start 235.7 103.89) (end 235.7 107.41) (width 0.1) (layer "F.Cu") (net 19))
+  (segment (start 265.92 99.77) (end 259.35 99.77) (width 0.1) (layer "F.Cu") (net 19))
+  (segment (start 235.7 107.41) (end 234.82 108.29) (width 0.1) (layer "F.Cu") (net 19))
+  (segment (start 259.93 99.4) (end 265.92 99.4) (width 0.1) (layer "F.Cu") (net 19))
+  (segment (start 259.35 99.77) (end 259.24 99.66) (width 0.1) (layer "F.Cu") (net 19))
+  (segment (start 268.28 100.11) (end 268.28 97.39) (width 0.1) (layer "F.Cu") (net 19))
+  (segment (start 267.27 97.2) (end 267.57 97.2) (width 0.1) (layer "F.Cu") (net 19))
+  (segment (start 233.55 108.79) (end 233.51 108.83) (width 0.1) (layer "F.Cu") (net 19))
+  (segment (start 245.01 99.79) (end 235.67 99.79) (width 0.1) (layer "F.Cu") (net 19))
+  (segment (start 259.24 99.11) (end 259.14 99.01) (width 0.1) (layer "F.Cu") (net 19))
+  (segment (start 267.74 97.37) (end 267.74 100.11) (width 0.1) (layer "F.Cu") (net 19))
+  (segment (start 234.29 108.29) (end 233.79 108.79) (width 0.1) (layer "F.Cu") (net 19))
+  (segment (start 245.28 99.01) (end 245.15 99.14) (width 0.1) (layer "F.Cu") (net 19))
+  (segment (start 266.25 99.01) (end 259.93 99.01) (width 0.1) (layer "F.Cu") (net 19))
+  (segment (start 235.67 99.79) (end 235.54 99.92) (width 0.1) (layer "F.Cu") (net 19))
+  (segment (start 272.07 96.82) (end 266.5 96.82) (width 0.1) (layer "F.Cu") (net 19))
+  (segment (start 266.39 98.87) (end 266.25 99.01) (width 0.1) (layer "F.Cu") (net 19))
+  (segment (start 245.15 99.65) (end 245.01 99.79) (width 0.1) (layer "F.Cu") (net 19))
   (segment (start 267.12 97.35) (end 267.27 97.2) (width 0.1) (layer "F.Cu") (net 19))
-  (segment (start 267.12 100.28) (end 267.12 97.35) (width 0.1) (layer "F.Cu") (net 19))
-  (segment (start 267.74 97.37) (end 267.74 100.11) (width 0.1) (layer "F.Cu") (net 19))
-  (segment (start 268.45 97.22) (end 272.12 97.22) (width 0.1) (layer "F.Cu") (net 19))
   (segment (start 266.27 104.01) (end 267.47 102.81) (width 0.1) (layer "F.Cu") (net 19))
+  (segment (start 235.54 99.92) (end 235.54 103.73) (width 0.1) (layer "F.Cu") (net 19))
+  (segment (start 245.15 99.14) (end 245.15 99.65) (width 0.1) (layer "F.Cu") (net 19))
+  (segment (start 267.47 100.63) (end 267.12 100.28) (width 0.1) (layer "F.Cu") (net 19))
+  (segment (start 266.27 104.68) (end 266.27 104.01) (width 0.1) (layer "F.Cu") (net 19))
+  (segment (start 259.14 99.01) (end 245.28 99.01) (width 0.1) (layer "F.Cu") (net 19))
   (segment (start 267.47 102.81) (end 267.47 100.63) (width 0.1) (layer "F.Cu") (net 19))
-  (segment (start 267.91 100.28) (end 268.11 100.28) (width 0.1) (layer "F.Cu") (net 19))
-  (segment (start 266.27 104.68) (end 266.27 104.01) (width 0.1) (layer "F.Cu") (net 19))
-  (segment (start 267.27 97.2) (end 267.57 97.2) (width 0.1) (layer "F.Cu") (net 19))
-  (segment (start 267.47 100.63) (end 267.12 100.28) (width 0.1) (layer "F.Cu") (net 19))
-  (segment (start 268.28 100.11) (end 268.28 97.39) (width 0.1) (layer "F.Cu") (net 19))
-  (segment (start 265.62 105.33) (end 266.27 104.68) (width 0.1) (layer "F.Cu") (net 19))
+  (segment (start 233.79 108.79) (end 233.55 108.79) (width 0.1) (layer "F.Cu") (net 19))
   (via (at 267.11 98.91) (size 0.56) (drill 0.3) (layers "F.Cu" "B.Cu") (net 19))
+  (arc (start 272.07 97.22) (mid 272.250253 97.022558) (end 272.07 96.82) (width 0.1) (layer "F.Cu") (net 19))
+  (arc (start 267.74 100.11) (mid 267.79 100.23) (end 267.91 100.28) (width 0.1) (layer "F.Cu") (net 19))
   (arc (start 268.11 100.28) (mid 268.23 100.23) (end 268.28 100.11) (width 0.1) (layer "F.Cu") (net 19))
-  (arc (start 267.74 100.11) (mid 267.79 100.23) (end 267.91 100.28) (width 0.1) (layer "F.Cu") (net 19))
-  (arc (start 267.74 97.37) (mid 267.69 97.25) (end 267.57 97.2) (width 0.1) (layer "F.Cu") (net 19))
-  (arc (start 268.45 97.22) (mid 268.33 97.27) (end 268.28 97.39) (width 0.1) (layer "F.Cu") (net 19))
+  (arc (start 265.92 99.4) (mid 266.100253 99.582558) (end 265.92 99.77) (width 0.1) (layer "F.Cu") (net 19))
+  (arc (start 259.93 99.01) (mid 259.749747 99.207442) (end 259.93 99.4) (width 0.1) (layer "F.Cu") (net 19))
+  (arc (start 268.28 97.39) (mid 268.33 97.27) (end 268.45 97.22) (width 0.1) (layer "F.Cu") (net 19))
+  (arc (start 267.57 97.2) (mid 267.69 97.25) (end 267.74 97.37) (width 0.1) (layer "F.Cu") (net 19))
 )

Commit message: route more traces
Connections:
- U2C1 pad F21: (no net) -> /CPU_D42
- U2C1 pad G20: (no net) -> /CPU_D49
- U2C1 pad G21: (no net) -> /CPU_D51
- U2C1 pad H19: (no net) -> /CPU_D44
- U4C1 pad A1: (no net) -> /CPU_D44
- U4C1 pad A2: (no net) -> /CPU_D51
- U4C1 pad A3: (no net) -> /CPU_D42
- U4C1 pad C3: (no net) -> /CPU_D49
Routing:
- net /CPU_D42: track 0.00 -> 80.6 mm, vias 0 -> 1
- net /CPU_D49: track 0.00 -> 80.3 mm, vias 0 -> 1
- net /CPU_D51: track 0.00 -> 78.5 mm, vias 0 -> 1
- net /CPU_D44: track 0.00 -> 78.3 mm, vias 0 -> 1

Commit message: route more traces
Connections:
- U2C1 pad AA11: (no net) -> /CPU_JTAG_TCK
- U2C1 pad AA14: (no net) -> /CPU_JTAG_TRST
- U2C1 pad AB20: (no net) -> /CPU_PREQ
- U2C1 pad AC15: (no net) -> /CPU_JTAG_TDO
- U2C1 pad AD13: (no net) -> /CPU_JTAG_TDI
- U2C1 pad AD14: (no net) -> /CPU_JTAG_TMS
- U2C1 pad H20: (no net) -> /VSS
- U2C1 pad H21: (no net) -> /CPU_D47
- U2C1 pad J19: (no net) -> /VSS
- U2C1 pad J20: (no net) -> /CPU_D46
- U2C1 pad J21: (no net) -> /CPU_D59
- U2C1 pad K18: (no net) -> /CPU_D52
- U2C1 pad K19: (no net) -> /CPU_D57
- U2C1 pad K20: (no net) -> /VSS
- U2C1 pad K21: (no net) -> /CPU_D53
- U2C1 pad L18: (no net) -> /CPU_D48
- U2C1 pad L19: (no net) -> /VSS
- U2C1 pad L20: (no net) -> /CPU_D60
- U2C1 pad L21: (no net) -> /CPU_D55
- U2C1 pad M18: (no net) -> /CPU_D54
- U2C1 pad M19: (no net) -> /CPU_D61
- U2C1 pad M20: (no net) -> /VSS
- U2C1 pad N18: (no net) -> /VSS
- U2C1 pad N19: (no net) -> /VSS
- U2C1 pad N20: (no net) -> /VSS
- U2C1 pad P17: (no net) -> /CPU_VCCT
- U2C1 pad P18: (no net) -> /CPU_D50
- U2C1 pad P19: (no net) -> /VSS
- U2C1 pad P20: (no net) -> /CPU_DEP6
- U2C1 pad P21: (no net) -> /CPU_DEP5
- U2C1 pad R17: (no net) -> /CPU_VCCT
- U2C1 pad R18: (no net) -> /CPU_D63
- U2C1 pad R19: (no net) -> /CPU_D56
- U2C1 pad R20: (no net) -> /VSS
- U2C1 pad R21: (no net) -> /CPU_DEP3
- U2C1 pad T17: (no net) -> /CPU_VCCT
- U2C1 pad T18: (no net) -> /VSS
- U2C1 pad T19: (no net) -> /VSS
- U2C1 pad T20: (no net) -> /CPU_D58
- U2C1 pad T21: (no net) -> /CPU_DEP1
- U2C1 pad U18: (no net) -> /CPU_D62
- U2C1 pad U19: (no net) -> /CPU_DEP7
- U2C1 pad U20: (no net) -> /VSS
- U2C1 pad U21: (no net) -> /CPU_DEP2
- U2C1 pad V10: (no net) -> /CPU_VCCT
- U2C1 pad V11: (no net) -> /CPU_VCCT
- U2C1 pad V12: (no net) -> /CPU_VCCT
- U2C1 pad V13: (no net) -> /CPU_VCCT
- U2C1 pad V14: (no net) -> /CPU_VCCT
- U2C1 pad V15: (no net) -> /CPU_VCCT
- U2C1 pad V16: (no net) -> /CPU_VCCT
- U2C1 pad V17: (no net) -> /CPU_VCCT
- U2C1 pad V18: (no net) -> /CPU_DEP4
- U2C1 pad V19: (no net) -> /VSS
- U2C1 pad V20: (no net) -> /CPU_DEP0
- U2C1 pad V21: (no net) -> /CPU_BINIT
- U2C1 pad V6: (no net) -> /CPU_VCCT
- U2C1 pad V7: (no net) -> /CPU_VCCT
- U2C1 pad V8: (no net) -> /CPU_VCCT
- U2C1 pad V9: (no net) -> /CPU_VCCT
- U4C1 pad B2: (no net) -> /CPU_D47
- U4C1 pad D1: (no net) -> /CPU_D55
- U4C1 pad E1: (no net) -> /CPU_D61
- U4C1 pad E2: (no net) -> /CPU_D58
- U4C1 pad E3: (no net) -> /CPU_D60
Routing:
- net /CPU_JTAG_TCK: track 0.00 -> 83.1 mm, vias 0 -> 1
- net /CPU_D60: track 0.00 -> 80.0 mm, vias 0 -> 1
- net /CPU_D61: track 0.00 -> 79.9 mm, vias 0 -> 1
- net /CPU_D58: track 0.00 -> 78.6 mm, vias 0 -> 1
- net /CPU_PREQ: track 0.00 -> 78.4 mm, vias 0 -> 1
- net /CPU_JTAG_TDI: track 0.00 -> 78.3 mm, vias 0 -> 1
- net /CPU_JTAG_TMS: track 0.00 -> 77.9 mm, vias 0 -> 1
- net /CPU_D47: track 0.00 -> 77.6 mm, vias 0 -> 1
- net /CPU_D55: track 0.00 -> 77.3 mm, vias 0 -> 1
- net /CPU_D46: track 0.00 -> 68.3 mm, vias 0 -> 1
- net /CPU_D59: track 0.00 -> 65.0 mm, vias 0 -> 1
- net /VSS: track 5.59 -> 18.2 mm, vias 5 -> 17
- net /CPU_DEP7: track 0.00 -> 9.36 mm, vias 0 -> 1
- net /CPU_DEP1: track 0.00 -> 8.16 mm, vias 0 -> 1
- net /CPU_DEP0: track 0.00 -> 5.36 mm, vias 0 -> 1
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
Commit message: route more
Connections:
- U2C1 pad B15: (no net) -> /VSS
- U2C1 pad B16: (no net) -> /CPU_D13
- U2C1 pad B17: (no net) -> /CPU_D22
- U2C1 pad C15: (no net) -> /VSS
- U2C1 pad C16: (no net) -> /VSS
- U2C1 pad C17: (no net) -> /CPU_D24
- U2C1 pad C18: (no net) -> /CPU_D26
- U2C1 pad D17: (no net) -> /CPU_D25
- U2C1 pad D18: (no net) -> /CPU_D28
- U2C1 pad E16: (no net) -> /CPU_VREF
- U2C1 pad E17: (no net) -> /CPU_VREF
- U2C1 pad F15: (no net) -> /VSS
- U2C1 pad F16: (no net) -> /VSS
- U2C1 pad F17: (no net) -> /CPU_VREF
- U4C1 pad A7: (no net) -> /CPU_D26
- U4C1 pad A8: (no net) -> /CPU_D22
- U4C1 pad B8: (no net) -> /CPU_D28
Routing:
- net /CPU_D26: track 0.00 -> 76.7 mm, vias 0 -> 1
- net /CPU_D22: track 0.00 -> 76.0 mm, vias 0 -> 1
- net /CPU_D28: track 0.00 -> 75.2 mm, vias 0 -> 1
- net /CPU_VREF: track 0.00 -> 3.05 mm, vias 0 -> 1
- net /VSS: track 18.2 -> 20.9 mm, vias 17 -> 18
- net /CPU_D25: track 0.00 -> 0.90 mm, vias 0 -> 1
- net /CPU_D24: track 0.00 -> 0.90 mm, vias 0 -> 1
- net /CPU_D13: track 0.00 -> 0.75 mm, vias 0 -> 1

Commit message: route more
Connections:
- U2C1 pad A14: (no net) -> /CPU_D10
- U2C1 pad B14: (no net) -> /CPU_D18
- U2C1 pad D15: (no net) -> /CPU_D16
- U2C1 pad E10: (no net) -> /VSS
- U2C1 pad E11: (no net) -> /VSS
- U2C1 pad E14: (no net) -> /CPU_D19
- U2C1 pad E7: (no net) -> /VSS
- U2C1 pad E8: (no net) -> /VSS
- U2C1 pad E9: (no net) -> /VSS
- U2C1 pad F10: (no net) -> /VSS
- U2C1 pad F11: (no net) -> /VSS
- U2C1 pad F12: (no net) -> /VSS
- U2C1 pad F13: (no net) -> /VSS
- U2C1 pad F14: (no net) -> /VSS
- U2C1 pad F6: (no net) -> /VSS
- U2C1 pad F7: (no net) -> /VSS
- U2C1 pad F8: (no net) -> /VSS
- U2C1 pad F9: (no net) -> /VSS
- U4C1 pad C9: (no net) -> /CPU_D18
Routing:
- net /CPU_D18: track 0.00 -> 79.8 mm, vias 0 -> 1
- net /VSS: track 20.9 -> 40.4 mm, vias 18 -> 21
- net /CPU_D10: track 0.00 -> 4.50 mm
- net /CPU_D19: track 0.00 -> 0.90 mm, vias 0 -> 1
- net /CPU_D16: track 0.00 -> 0.88 mm, vias 0 -> 1

Commit message: route more
Connections:
- U2C1 pad A12: (no net) -> /VSS
- U2C1 pad A13: (no net) -> /CPU_D14
- U2C1 pad B10: (no net) -> /VSS
- U2C1 pad B11: (no net) -> /CPU_D7
- U2C1 pad B12: (no net) -> /CPU_D11
- U2C1 pad B13: (no net) -> /CPU_D9
- U2C1 pad B9: (no net) -> /CPU_D4
- U2C1 pad C10: (no net) -> /CPU_D6
- U2C1 pad C11: (no net) -> /VSS
- U2C1 pad C12: (no net) -> /CPU_D8
- U2C1 pad C13: (no net) -> /CPU_D20
- U2C1 pad C9: (no net) -> /VSS
- U2C1 pad D10: (no net) -> /CPU_D0
- U2C1 pad D11: (no net) -> /CPU_D1
- U2C1 pad D12: (no net) -> /CPU_D17
- U2C1 pad D13: (no net) -> /CPU_D15
- U2C1 pad D9: (no net) -> /VSS
- U2C1 pad E12: (no net) -> /CPU_D12
- U2C1 pad E13: (no net) -> /VSS
- U4C1 pad A10: (no net) -> /CPU_D9
- U4C1 pad A11: (no net) -> /CPU_D20
- U4C1 pad A12: (no net) -> /CPU_D6
- U4C1 pad A13: (no net) -> /CPU_D0
- U4C1 pad A9: (no net) -> /CPU_D10
- U4C1 pad B10: (no net) -> /CPU_D14
- U4C1 pad B12: (no net) -> /CPU_D7
Routing:
- net /CPU_D9: track 0.00 -> 76.1 mm, vias 0 -> 1
- net /CPU_D7: track 0.00 -> 76.1 mm, vias 0 -> 1
- net /CPU_D6: track 0.00 -> 75.8 mm, vias 0 -> 1
- net /CPU_D14: track 0.00 -> 75.6 mm, vias 0 -> 1
- net /CPU_D0: track 0.00 -> 75.3 mm, vias 0 -> 1
- net /CPU_D20: track 0.00 -> 74.9 mm, vias 0 -> 1
- net /CPU_D10: track 4.50 -> 76.8 mm, vias 0 -> 1
- net /VSS: track 40.4 -> 46.2 mm, vias 21 -> 25
- net /CPU_D12: track 0.00 -> 0.91 mm, vias 0 -> 1
- net /CPU_D1: track 0.00 -> 0.88 mm, vias 0 -> 1
- net /CPU_D8: track 0.00 -> 0.88 mm, vias 0 -> 1
- net /CPU_D15: track 0.00 -> 0.87 mm, vias 0 -> 1
- net /CPU_D11: track 0.00 -> 0.87 mm, vias 0 -> 1
- net /CPU_D17: track 0.00 -> 0.86 mm, vias 0 -> 1
